Commit message: Split kingfisher_gazebo out of kingfisher_description
kingfisher_description is now Gazebo-free: links, joints, meshes and a
new kingfisher.urdf.xacro top level for robot_state_publisher. Its
package.xml drops wamv_gazebo / vrx_gazebo, so it can move to the
kingfisher repo without pulling ros_gz into the boat build.

kingfisher_gazebo holds everything else: the VRX hydrodynamics and
thruster plugins, preserveFixedJoint, the <sensor> blocks and the
kingfisher_gazebo.urdf.xacro top level, which includes
kingfisher.urdf.xacro. Sensor poses now live only in the description;
the *_enabled args gate the Gazebo sensor, not the link.

The lidar sensor comes from the planar_lidar_2d macro that was patched
into src/vrx (untracked), folded into kingfisher_sensors_gazebo.xacro so
nothing in the xacro chain references wamv_gazebo any more.

Checked: the generated URDF and `gz sdf -p` output match the pre-split
ones element for element (order aside), and kingfisher.urdf.xacro runs
with no VRX package on the path.

Source: vrx (upstream jazzy, untracked) vrx_urdf/wamv_gazebo/urdf/components/planar_lidar_2d.xacro

Co-Authored-By: Claude Opus 5.5 <noreply@anthropic.com>

File: kingfisher_description/urdf/kingfisher_base.urdf.xacro (robot description, xacro)
@@ -28,5 +28,5 @@
 a TF prefix is added by robot_state_publisher (frame_prefix), never baked into
 the URDF. Hull dynamics are provided by the VRX Surface / SimpleHydrodynamics
-plugins (see kingfisher_gazebo_plugins.xacro).
+plugins (see kingfisher_gazebo).
 Frame convention (base_link, x forward, z up): the hull mesh spans
 x -0.64..0.70, y +-0.49, z -0.22..0.10; keel at z = -0.22.

File: kingfisher_description/urdf/kingfisher_sensors.xacro (robot description, xacro)
@@ -1,12 +1,8 @@
 <?xml version="1.0"?>
 <!--
-Sensor macros for the Kingfisher M200.
+Sensor links of the Kingfisher M200.
 Every macro creates a plainly named link (<name>_link) on a fixed joint to
-base_link and a Gazebo sensor whose published frame_id is forced with
-<gz_frame_id> to ${tf_prefix}<name>_link, i.e. the same frame the real driver
-would stamp and the same frame robot_state_publisher publishes (frame_prefix).
-Gazebo lumps the fixed-joint links into base_link internally, which does not
-matter: TF comes from the URDF via robot_state_publisher, not from Gazebo.
-Requires the global properties tf_prefix and sensor_namespace.
+base_link. The Gazebo sensors attached to these links are in
+kingfisher_gazebo/urdf/kingfisher_sensors_gazebo.xacro.
 -->
 <robot xmlns:xacro="http://ros.org/wiki/xacro">
@@ -41,59 +37,20 @@
     </joint>
   </xacro:macro>
-  <!-- GPS receiver: sensor "navsat" -> sensors/gps/gps/fix -->
-  <xacro:macro name="kingfisher_gps" params="name:=gps x:=0 y:=0 z:=0 R:=0 P:=0 Y:=0 update_rate:=20">
+  <xacro:macro name="kingfisher_gps" params="name:=gps x:=0 y:=0 z:=0 R:=0 P:=0 Y:=0">
     <xacro:kingfisher_sensor_link name="${name}" xyz="${x} ${y} ${z}" rpy="${R} ${P} ${Y}"
                                   radius="0.04" length="0.03" mass="0.2"/>
-    <gazebo reference="${name}_link">
-      <sensor name="navsat" type="navsat">
-        <always_on>1</always_on>
-        <update_rate>${update_rate}</update_rate>
-        <gz_frame_id>${tf_prefix}${name}_link</gz_frame_id>
-      </sensor>
-    </gazebo>
   </xacro:macro>
-  <!-- Gaussian noise block of the gz IMU sensor -->
-  <xacro:macro name="kf_imu_noise" params="stddev bias_mean bias_stddev dyn_bias_stddev dyn_bias_time precision">
-    <noise type="gaussian">
-      <mean>0</mean>
-      <stddev>${stddev}</stddev>
-      <bias_mean>${bias_mean}</bias_mean>
-      <bias_stddev>${bias_stddev}</bias_stddev>
-      <dynamic_bias_stddev>${dyn_bias_stddev}</dynamic_bias_stddev>
-      <dynamic_bias_correlation_time>${dyn_bias_time}</dynamic_bias_correlation_time>
-      <precision>${precision}</precision>
-    </noise>
-  </xacro:macro>
-  <!-- IMU: sensor "<name>_sensor" -> sensors/imu/imu/data (noise model as the WAM-V's) -->
-  <xacro:macro name="kingfisher_imu" params="name:=imu x:=0 y:=0 z:=0 R:=0 P:=0 Y:=0 update_rate:=100">
+  <xacro:macro name="kingfisher_imu" params="name:=imu x:=0 y:=0 z:=0 R:=0 P:=0 Y:=0">
     <xacro:kingfisher_sensor_link name="${name}" xyz="${x} ${y} ${z}" rpy="${R} ${P} ${Y}"
                                   radius="0.02" length="0.01" mass="0.05"/>
-    <gazebo reference="${name}_link">
-      <sensor type="imu" name="${name}_sensor">
-        <update_rate>${update_rate}</update_rate>
-        <gz_frame_id>${tf_prefix}${name}_link</gz_frame_id>
-        <imu>
-          <angular_velocity>
-            <x><xacro:kf_imu_noise stddev="0.009" bias_mean="0.00075" bias_stddev="0.005" dyn_bias_stddev="0.00002" dyn_bias_time="400.0" precision="0.00025"/></x>
-            <y><xacro:kf_imu_noise stddev="0.009" bias_mean="0.00075" bias_stddev="0.005" dyn_bias_stddev="0.00002" dyn_bias_time="400.0" precision="0.00025"/></y>
-            <z><xacro:kf_imu_noise stddev="0.009" bias_mean="0.00075" bias_stddev="0.005" dyn_bias_stddev="0.00002" dyn_bias_time="400.0" precision="0.00025"/></z>
-          </angular_velocity>
-          <linear_acceleration>
-            <x><xacro:kf_imu_noise stddev="0.021" bias_mean="0.05" bias_stddev="0.0075" dyn_bias_stddev="0.000375" dyn_bias_time="175.0" precision="0.005"/></x>
-            <y><xacro:kf_imu_noise stddev="0.021" bias_mean="0.05" bias_stddev="0.0075" dyn_bias_stddev="0.000375" dyn_bias_time="175.0" precision="0.005"/></y>
-            <z><xacro:kf_imu_noise stddev="0.021" bias_mean="0.05" bias_stddev="0.0075" dyn_bias_stddev="0.000375" dyn_bias_time="175.0" precision="0.005"/></z>
-          </linear_acceleration>
-          <orientation_reference_frame>
-            <localization>ENU</localization>
-          </orientation_reference_frame>
-        </imu>
-      </sensor>
-    </gazebo>
   </xacro:macro>
-  <!-- Monocular camera: sensor "<name>_sensor" -> sensors/cameras/<name>_sensor/{image_raw,camera_info}.
-       <name>_link is the camera body (x forward, z up), <name>_link_optical the
-       REP 103 optical frame (z forward) that the images are stamped with. -->
-  <xacro:macro name="kingfisher_camera" params="name:=camera x:=0 y:=0 z:=0 R:=0 P:=0 Y:=0
-                                                width:=1280 height:=720 hfov:=1.3962634 update_rate:=30 visualize:=false">
+  <!-- 2D lidar, sized as a SICK TiM571 -->
+  <xacro:macro name="kingfisher_lidar" params="name:=lidar x:=0 y:=0 z:=0 R:=0 P:=0 Y:=0">
+    <xacro:kingfisher_sensor_link name="${name}" xyz="${x} ${y} ${z}" rpy="${R} ${P} ${Y}"
+                                  radius="0.03" length="0.086" mass="0.25"/>
+  </xacro:macro>
+  <!-- Monocular camera. <name>_link is the camera body (x forward, z up),
+       <name>_link_optical the REP 103 optical frame (z forward). -->
+  <xacro:macro name="kingfisher_camera" params="name:=camera x:=0 y:=0 z:=0 R:=0 P:=0 Y:=0">
     <xacro:kingfisher_sensor_link name="${name}" xyz="${x} ${y} ${z}" rpy="${R} ${P} ${Y}"
                                   radius="0.02" length="0.04" mass="0.1"/>
@@ -104,28 +61,4 @@
       <child link="${name}_link_optical"/>
     </joint>
-    <gazebo reference="${name}_link">
-      <sensor type="camera" name="${name}_sensor">
-        <update_rate>${update_rate}</update_rate>
-        <visualize>${visualize}</visualize>
-        <gz_frame_id>${tf_prefix}${name}_link_optical</gz_frame_id>
-        <camera name="${name}_camera">
-          <horizontal_fov>${hfov}</horizontal_fov>
-          <image>
-            <width>${width}</width>
-            <height>${height}</height>
-            <format>R8G8B8</format>
-          </image>
-          <clip>
-            <near>0.05</near>
-            <far>400</far>
-          </clip>
-          <noise>
-            <type>gaussian</type>
-            <mean>0.0</mean>
-            <stddev>0.007</stddev>
-          </noise>
-        </camera>
-      </sensor>
-    </gazebo>
   </xacro:macro>
 </robot>

File: kingfisher_description/urdf/kingfisher_thruster.xacro (robot description, xacro)
@@ -5,5 +5,5 @@
 continuous joint named ${prefix}_engine_propeller_joint, which is
 the joint driven by gz::sim::systems::Thruster (see
-kingfisher_gazebo_plugins.xacro). The propeller joint name follows the WAM-V
+kingfisher_gazebo). The propeller joint name follows the WAM-V
 convention (<prefix>_engine_propeller_joint) so the VRX bridge generation
 works unchanged.
@@ -46,8 +46,4 @@
       <child link="${prefix}_thruster_link"/>
     </joint>
-    <!-- Keep the housing as its own link instead of lumping it into base_link -->
-    <gazebo reference="${prefix}_base_thruster_joint">
-      <preserveFixedJoint>true</preserveFixedJoint>
-    </gazebo>
     <!-- Propeller / impeller, spins about x -->
     <link name="${prefix}_propeller_link">

File: kingfisher_gazebo/urdf/kingfisher_gazebo.urdf.xacro (robot description, xacro)
@@ -1,5 +1,6 @@
 <?xml version="1.0"?>
 <!--
-Top-level Kingfisher M200 description for VRX / gz-sim.
+Top-level Kingfisher M200 for VRX / gz-sim: kingfisher_description's
+kingfisher.urdf.xacro plus the Gazebo plugins and sensors.
 This is the file vrx_gz processes (xacro -> URDF -> gz sdf -p). vrx_gz always
 passes namespace:=<model_name> locked:=true vrx_sensors_enabled:=true
@@ -22,5 +23,6 @@
   <!-- Standard sensor suite: GPS, IMU, 2D lidar, front camera -->
   <xacro:arg name="vrx_sensors_enabled" default="true"/>
-  <!-- Individual sensors (used when vrx_sensors_enabled is false) -->
+  <!-- Individual sensors (used when vrx_sensors_enabled is false). The links
+       always exist; these only toggle the Gazebo sensor. -->
   <xacro:arg name="camera_enabled" default="false"/>
   <xacro:arg name="gps_enabled" default="false"/>
@@ -37,8 +39,7 @@
   <xacro:property name="sensor_namespace" value="$(arg sensor_namespace)" scope="global"/>
   <!-- === Platform === -->
-  <xacro:include filename="$(find kingfisher_description)/urdf/kingfisher_base.urdf.xacro"/>
-  <xacro:include filename="$(find kingfisher_description)/urdf/kingfisher_gazebo_plugins.xacro"/>
-  <xacro:include filename="$(find kingfisher_description)/urdf/kingfisher_sensors.xacro"/>
-  <xacro:include filename="$(find wamv_gazebo)/urdf/components/planar_lidar_2d.xacro"/>
+  <xacro:include filename="$(find kingfisher_description)/urdf/kingfisher.urdf.xacro"/>
+  <xacro:include filename="$(find kingfisher_gazebo)/urdf/kingfisher_gazebo_plugins.xacro"/>
+  <xacro:include filename="$(find kingfisher_gazebo)/urdf/kingfisher_sensors_gazebo.xacro"/>
   <!-- === Dynamics and propulsion === -->
   <xacro:kingfisher_dynamics_gazebo/>
@@ -70,6 +71,5 @@
     </gazebo>
   </xacro:if>
-  <!-- === Sensors === -->
-  <!-- Deck is at z ~0.05-0.10, bow at x ~0.70 -->
+  <!-- === Sensors (links and poses are in kingfisher.urdf.xacro) === -->
   <xacro:property name="kf_true" value="${['true', '1']}"/>
   <xacro:property name="kf_all" value="${'$(arg vrx_sensors_enabled)'.lower() in kf_true}"/>
@@ -79,15 +79,14 @@
   <xacro:property name="kf_imu" value="${kf_all or '$(arg imu_enabled)'.lower() in kf_true}"/>
   <xacro:if value="${kf_lidar}">
-    <xacro:planar_lidar_2d name="lidar" x="0.30" y="0" z="0.35"
-                           link_prefix="" frame_id="${tf_prefix}lidar_link"/>
+    <xacro:kingfisher_lidar_gazebo name="lidar"/>
   </xacro:if>
   <xacro:if value="${kf_camera}">
-    <xacro:kingfisher_camera name="camera" x="0.55" y="0" z="0.25" P="${radians(10)}"/>
+    <xacro:kingfisher_camera_gazebo name="camera"/>
   </xacro:if>
   <xacro:if value="${kf_gps}">
-    <xacro:kingfisher_gps name="gps" x="-0.30" y="0" z="0.30"/>
+    <xacro:kingfisher_gps_gazebo name="gps"/>
   </xacro:if>
   <xacro:if value="${kf_imu}">
-    <xacro:kingfisher_imu name="imu" x="0" y="0" z="0.05"/>
+    <xacro:kingfisher_imu_gazebo name="imu"/>
   </xacro:if>
 </robot>

File: kingfisher_gazebo/urdf/kingfisher_gazebo_plugins.xacro (robot description, xacro)
@@ -95,4 +95,8 @@
   </xacro:macro>
   <xacro:macro name="kingfisher_thruster_plugin" params="name">
+    <!-- Keep the housing as its own link instead of lumping it into base_link -->
+    <gazebo reference="${name}_base_thruster_joint">
+      <preserveFixedJoint>true</preserveFixedJoint>
+    </gazebo>
     <gazebo>
       <plugin filename="gz-sim-thruster-system" name="gz::sim::systems::Thruster">
