Commit message: Drop the unused thruster_namespace and sensor_namespace xacro args
Both were copied from wamv_gazebo.urdf.xacro, and nothing reads them.
vrx_gz never passes them, and its bridges hardcode
thrusters/<name>/thrust and sensors/<kind>/..., so setting one would only
move the gz topic off the bridge and the thrusters would get no command.
locked and thruster_config stay because vrx_gz passes them.

Checked: the generated URDF is byte-identical before and after.

Co-Authored-By: Claude Opus 5.5 <noreply@anthropic.com>

File: kingfisher_gazebo/urdf/kingfisher_gazebo.urdf.xacro (robot description, xacro)
@@ -31,11 +31,6 @@
   <!-- Ground truth odometry message on sensors/position/ground_truth_odometry (no TF) -->
   <xacro:arg name="ground_truth_enabled" default="true"/>
-  <!-- Topic sub-namespaces -->
-  <xacro:arg name="thruster_namespace" default="thrusters/"/>
-  <xacro:arg name="sensor_namespace" default="sensors/"/>
   <xacro:property name="namespace" value="$(arg namespace)" scope="global"/>
   <xacro:property name="tf_prefix" value="$(arg tf_prefix)" scope="global"/>
-  <xacro:property name="thruster_namespace" value="$(arg thruster_namespace)" scope="global"/>
-  <xacro:property name="sensor_namespace" value="$(arg sensor_namespace)" scope="global"/>
   <!-- === Platform === -->
   <xacro:include filename="$(find kingfisher_description)/urdf/kingfisher.urdf.xacro"/>

Commit message: Add sail actuation to the sim
The sail turns on sail_joint through a JointPositionController in
velocity mode, the way the WAM-V's steerable thrusters do: each step it
sets the joint velocity towards the target, capped by <cmd_max>, so the
sail turns at kf_sail_max_speed (1.0 rad/s, a placeholder until the real
stepper is measured) and then holds rigidly. The plugin's <name>sail</name>
makes vrx_gz bridge ROS thrusters/sail/pos to it, with no VRX change.

robot.launch.py adds the sim side of the sail interface:
- sail/cmd_angle: the absolute sail_joint angle in rad, 0 along the
  hull, + counter-clockwise from above, reported in joint_states.
  sail_relay (topic_tools relay) forwards it to thrusters/sail/pos.
- sail/cmd_rate: rad/s, for jogging. sail_jog walks the angle target
  from the measured angle at that rate, clamped to max_rate, and sets it
  to the measured angle when the rate goes to zero or stops for
  1/min_rate (0.1 s), so the sail stops where it is. The boat's sail
  controller may offer this natively; that is decided with the boat
  side of the sail.

Co-Authored-By: Claude Opus 5.5 <noreply@anthropic.com>

File: kingfisher_gazebo/urdf/kingfisher_gazebo.urdf.xacro (robot description, xacro)
@@ -41,4 +41,6 @@
   <xacro:kingfisher_thruster_plugin name="left"/>
   <xacro:kingfisher_thruster_plugin name="right"/>
+  <!-- ROS thrusters/sail/pos; robot.launch.py relays sail/cmd_angle to it -->
+  <xacro:kingfisher_sail_plugin/>
   <!-- === Joint states (propeller spin), bridged to joint_states for robot_state_publisher === -->
   <gazebo>

File: kingfisher_gazebo/urdf/kingfisher_gazebo_plugins.xacro (robot description, xacro)
@@ -2,6 +2,6 @@
 <!--
 gz-sim plugins for the Kingfisher M200: hull buoyancy (vrx::Surface, one per
-hull), Fossen drag (vrx::SimpleHydrodynamics) and one gz::sim::systems::Thruster
-per jet drive.
+hull), Fossen drag (vrx::SimpleHydrodynamics), one gz::sim::systems::Thruster
+per jet drive, and a JointPositionController that turns the sail.
 Hydrodynamic coefficients come from the system identification used in the
 IsaacLab kingfisher environment (linear / quadratic damping, body frame):
@@ -115,3 +115,22 @@
     </gazebo>
   </xacro:macro>
+  <!-- === Sail === -->
+  <!-- rad/s; placeholder until the real stepper is measured -->
+  <xacro:property name="kf_sail_max_speed" value="1.0"/>
+  <!-- Velocity mode: turns sail_joint at kf_sail_max_speed to the commanded
+       angle, then holds it rigidly, like a stepper -->
+  <xacro:macro name="kingfisher_sail_plugin">
+    <gazebo>
+      <plugin filename="gz-sim-joint-position-controller-system"
+              name="gz::sim::systems::JointPositionController">
+        <joint_name>sail_joint</joint_name>
+        <use_velocity_commands>true</use_velocity_commands>
+        <cmd_max>${kf_sail_max_speed}</cmd_max>
+        <topic>${namespace}/thrusters/sail/pos</topic>
+        <!-- Not used by Gazebo; vrx_gz bridges thrusters/<name>/pos from it.
+             Required: vrx_gz fails without it. -->
+        <name>sail</name>
+      </plugin>
+    </gazebo>
+  </xacro:macro>
 </robot>

Commit message: Add ApparentWind: sail lift and drag and a 2D anemometer
A gz model system in kingfisher_gazebo, loaded from the xacro next to the
thruster and sail plugins. It reads the true wind from vrx::USVWind's
/vrx/debug/wind/{speed,direction} (zero until they publish) and uses the
apparent wind, the true wind minus the velocity of the point:

- Sail: lift and drag from a NACA 0018 table, F = qA [C_D u + C_L (z x u)],
  with the angle of attack from the chord's nose to where the wind comes
  from. Applied at center_of_effort (the sail_link origin for now) with
  Link::AddWorldWrench: Link::AddWorldForce(F, p) offsets from the centre
  of mass, which is 0.35 m above the sail_link origin. The force in
  sail_link goes out on /<ns>/sail/wrench at 20 Hz.
- Anemometer: the apparent wind at anemometer_link, in that frame (FRD),
  z dropped, through a first-order low-pass (tau 1 s, a placeholder), on
  /<ns>/sensors/anemometer/twist (gz.msgs.Twist, linear) at 10 Hz. The
  frame's pose is resolved from the model's SDF DOM, so the description
  stays the only source of geometry.

Stamps are sim time, and frame ids carry the tf prefix.

The table is the Re 80,000 NACA 0018 data over 0-180 deg from Sheldahl &
Klimas, "Aerodynamic Characteristics of Seven Symmetrical Airfoil
Sections Through 180-Degree Angle of Attack for Use in Aerodynamic
Analysis of Vertical Axis Wind Turbines", SAND80-2114, Sandia, 1981, as
tabulated in Sandia's CACTUS (test/Airfoil_Section_Data/NACA_0018.dat,
identical to the copy in OWENS.jl). It is used as published, with no
finite-span correction. The values are placeholders until the boat logs.

WindModel.hh holds the table lookup, the sail force and the filter,
header-only so test_wind_model can check them: the sign checks, mirror
symmetry, interpolation and the filter's step response.

A hook puts lib/ on GZ_SIM_SYSTEM_PLUGIN_PATH.

Co-Authored-By: Claude Opus 5.5 <noreply@anthropic.com>

File: kingfisher_gazebo/urdf/kingfisher_gazebo.urdf.xacro (robot description, xacro)
@@ -43,4 +43,6 @@
   <!-- ROS thrusters/sail/pos; robot.launch.py relays sail/cmd_angle to it -->
   <xacro:kingfisher_sail_plugin/>
+  <!-- Sail aero force and the anemometer, from USVWind's wind -->
+  <xacro:kingfisher_wind_plugin/>
   <!-- === Joint states (propeller spin), bridged to joint_states for robot_state_publisher === -->
   <gazebo>

File: kingfisher_gazebo/urdf/kingfisher_gazebo_plugins.xacro (robot description, xacro)
@@ -3,5 +3,6 @@
 gz-sim plugins for the Kingfisher M200: hull buoyancy (vrx::Surface, one per
 hull), Fossen drag (vrx::SimpleHydrodynamics), one gz::sim::systems::Thruster
-per jet drive, and a JointPositionController that turns the sail.
+per jet drive, a JointPositionController that turns the sail, and
+kingfisher_gazebo::ApparentWind for the sail's aero force and the anemometer.
 Hydrodynamic coefficients come from the system identification used in the
 IsaacLab kingfisher environment (linear / quadratic damping, body frame):
@@ -134,3 +135,57 @@
     </gazebo>
   </xacro:macro>
+  <!-- === Wind: sail aero force and anemometer === -->
+  <!-- m^2: span 0.70 x chord 0.20 -->
+  <xacro:property name="kf_sail_area" value="0.14"/>
+  <!-- Point of application in sail_link -->
+  <xacro:property name="kf_sail_ce" value="0 0 0"/>
+  <!-- NACA 0018, Re 80k (Sheldahl & Klimas 1981), 0-180 deg; mirrored for negative angles -->
+  <xacro:property name="kf_sail_alpha" value="
+    0 1 2 3 4 5 6 7 8 9 10 11 12
+    14 16 18 20 22 25 30 35 40 45 50 55 60
+    65 70 75 80 85 90 95 100 105 110 115 120 125
+    130 135 140 145 150 155 160 165 170 175 180"/>
+  <xacro:property name="kf_sail_cl" value="
+    0 0.0889 0.1935 0.2924 0.388 0.4753 0.5615 0.6224 0.6589 0.6606 0.6248 0.5531 0.4408
+    0.2256 0.2027 0.2603 0.3472 0.443 0.5963 0.855 0.98 1.035 1.05 1.02 0.955 0.875
+    0.76 0.63 0.5 0.365 0.23 0.09 -0.05 -0.185 -0.32 -0.45 -0.575 -0.67 -0.76
+    -0.85 -0.93 -0.98 -0.9 -0.77 -0.67 -0.635 -0.68 -0.85 -0.66 0"/>
+  <xacro:property name="kf_sail_cd" value="
+    0.0162 0.0163 0.0167 0.0172 0.0181 0.0192 0.0206 0.0223 0.0242 0.0264 0.0288 0.0315 0.08
+    0.158 0.196 0.238 0.282 0.329 0.405 0.57 0.745 0.92 1.075 1.215 1.345 1.47
+    1.575 1.665 1.735 1.78 1.8 1.8 1.78 1.75 1.7 1.635 1.555 1.465 1.35
+    1.225 1.085 0.925 0.755 0.575 0.42 0.32 0.23 0.14 0.055 0.025"/>
+  <!-- s; first-order low-pass on the anemometer reading. Placeholder. -->
+  <xacro:property name="kf_anemometer_tau" value="1.0"/>
+  <!-- Apparent wind = vrx::USVWind's true wind - the point's velocity.
+       Publishes sail/wrench (gz.msgs.Wrench) and sensors/anemometer/twist
+       (gz.msgs.Twist, linear = the 2D reading); robot.launch.py bridges them. -->
+  <xacro:macro name="kingfisher_wind_plugin">
+    <gazebo>
+      <plugin filename="libApparentWind.so" name="kingfisher_gazebo::ApparentWind">
+        <!-- USVWind's topics; zero wind until they publish -->
+        <topic_wind_speed>/vrx/debug/wind/speed</topic_wind_speed>
+        <topic_wind_direction>/vrx/debug/wind/direction</topic_wind_direction>
+        <sail>
+          <link_name>sail_link</link_name>
+          <center_of_effort>${kf_sail_ce}</center_of_effort>
+          <area>${kf_sail_area}</area>
+          <air_density>1.225</air_density>
+          <alpha>${kf_sail_alpha}</alpha>
+          <cl>${kf_sail_cl}</cl>
+          <cd>${kf_sail_cd}</cd>
+          <topic>/${namespace}/sail/wrench</topic>
+          <frame_id>${tf_prefix}sail_link</frame_id>
+          <rate>20</rate>
+        </sail>
+        <anemometer>
+          <frame>anemometer_link</frame>
+          <time_constant>${kf_anemometer_tau}</time_constant>
+          <topic>/${namespace}/sensors/anemometer/twist</topic>
+          <frame_id>${tf_prefix}anemometer_link</frame_id>
+          <rate>10</rate>
+        </anemometer>
+      </plugin>
+    </gazebo>
+  </xacro:macro>
 </robot>
