Commit message: Drive the sail using kingfisher_sail's sail_controller
The sim runs the boat's sail_controller with kingfisher.yaml.
sail_stepper_sim stands in for the Phidgets stepper:
- takes phidgets_stepper/command (STEP, RUN) and ramps the position at
  the stepper's acceleration (10 rad/s^2, read from kingfisher.yaml);
- publishes it on thrusters/sail/pos;
- publishes sail/calibrated: true once (latched). Calibration stays
  boat-only.

sail_jog, sail_relay and config/sail_jog.yaml are removed.
kf_sail_max_speed goes from 1.0 to 3.0, a cap above the stepper's
2.0 rad/s, so the joint follows the ramped positions.

robot.launch.py also starts joy_teleop with kingfisher_teleop's config
(arg teleop, default True, passed through by kingfisher_sim.launch.py),
as the boat bringup does.

kingfisher_sim exec_depends on kingfisher_sail, phidgets_msgs,
kingfisher_teleop and joy_teleop.

File: kingfisher_gazebo/urdf/kingfisher_gazebo.urdf.xacro (robot description, xacro)
@@ -41,5 +41,5 @@
   <xacro:kingfisher_thruster_plugin name="left"/>
   <xacro:kingfisher_thruster_plugin name="right"/>
-  <!-- ROS thrusters/sail/pos; robot.launch.py relays sail/cmd_angle to it -->
+  <!-- ROS thrusters/sail/pos, from sail_stepper_sim (robot.launch.py) -->
   <xacro:kingfisher_sail_plugin/>
   <!-- Sail aero force and the anemometer, from USVWind's wind -->

File: kingfisher_gazebo/urdf/kingfisher_gazebo_plugins.xacro (robot description, xacro)
@@ -117,8 +117,9 @@
   </xacro:macro>
   <!-- === Sail === -->
-  <!-- rad/s; placeholder until the real stepper is measured -->
-  <xacro:property name="kf_sail_max_speed" value="1.0"/>
-  <!-- Velocity mode: turns sail_joint at kf_sail_max_speed to the commanded
-       angle, then holds it rigidly, like a stepper -->
+  <!-- rad/s; only a cap above the stepper's 2.0 (sail_controller max_velocity),
+       so the controller follows sail_stepper_sim's ramped positions -->
+  <xacro:property name="kf_sail_max_speed" value="3.0"/>
+  <!-- Velocity mode: turns sail_joint at up to kf_sail_max_speed to the
+       commanded angle, then holds it rigidly, like a stepper -->
   <xacro:macro name="kingfisher_sail_plugin">
     <gazebo>
