Commit message: Publish the sim anemometer in base_link at the Rowind's rate
The anemometer contract moved to kingfisher/base_link (FLU), which is what
the boat's rowind7 driver now publishes. ApparentWind gets <output_frame>:
the reading is still computed in the anemometer frame (z dropped, then
low-passed) and is rotated into the output frame before publishing, in the
same order as the driver. The output frame may be a link (base_link) or a
frame of the model. The rotation follows the description, where
anemometer_link is yawed by pi (the real sensor's bow mark points aft), so
the sim and the boat agree on the mount.

The rate is 1.875 Hz, measured from the boat's Rowind 7 (kf_anemometer_rate).
The boat publishes unfiltered; the sim's tau = 1 s stays as a placeholder.

Co-Authored-By: Claude Opus 5.5 <noreply@anthropic.com>

File: kingfisher_gazebo/urdf/kingfisher_gazebo_plugins.xacro (robot description, xacro)
@@ -159,4 +159,6 @@
   <!-- s; first-order low-pass on the anemometer reading. Placeholder. -->
   <xacro:property name="kf_anemometer_tau" value="1.0"/>
+  <!-- Hz; the boat's Rowind 7, measured 2026-10-13 -->
+  <xacro:property name="kf_anemometer_rate" value="1.875"/>
   <!-- Apparent wind = vrx::USVWind's true wind - the point's velocity.
        Publishes sail/wrench (gz.msgs.Wrench) and sensors/anemometer/twist
@@ -182,8 +184,10 @@
         <anemometer>
           <frame>anemometer_link</frame>
+          <!-- The reading is rotated into this, as the boat's driver does -->
+          <output_frame>base_link</output_frame>
           <time_constant>${kf_anemometer_tau}</time_constant>
           <topic>/${namespace}/sensors/anemometer/twist</topic>
-          <frame_id>${tf_prefix}anemometer_link</frame_id>
-          <rate>10</rate>
+          <frame_id>${tf_prefix}base_link</frame_id>
+          <rate>${kf_anemometer_rate}</rate>
         </anemometer>
       </plugin>
